Commit message: Fix Panda gripper mimic controller setup

File: mcg5353_panda_gazebo_moveit/config/panda_gazebo.urdf.xacro (robot description, xacro)
@@ -283,5 +283,5 @@
         <axis xyz="0 -1 0" />
         <limit effort="20" lower="0.0" upper="0.04" velocity="0.2" />
-        <mimic joint="panda_finger_joint1" />
+        <mimic joint="panda_finger_joint1" multiplier="1.0" offset="0.0"/>
     </joint>
     <gazebo reference="panda_link0">
@@ -311,5 +311,22 @@
         <xacro:gazebo_position_joint joint_name="panda_joint6" initial_value="1.571"/>
         <xacro:gazebo_position_joint joint_name="panda_joint7" initial_value="0.785"/>
-        <xacro:gazebo_position_joint joint_name="panda_finger_joint1" initial_value="0.04"/>
+        <joint name="panda_finger_joint1">
+            <command_interface name="position"/>
+            <state_interface name="position">
+                <param name="initial_value">0.04</param>
+            </state_interface>
+            <state_interface name="velocity"/>
+            <state_interface name="effort"/>
+        </joint>
+        <joint name="panda_finger_joint2">
+            <param name="mimic">panda_finger_joint1</param>
+            <param name="multiplier">1</param>
+            <command_interface name="position"/>
+            <state_interface name="position">
+                <param name="initial_value">0.04</param>
+            </state_interface>
+            <state_interface name="velocity"/>
+            <state_interface name="effort"/>
+        </joint>
     </ros2_control>
     <gazebo>

Commit message: Finger mimic fixed.

File: mcg5353_panda_gazebo_moveit/config/panda_gazebo.urdf.xacro (robot description, xacro)
@@ -275,5 +275,5 @@
         <origin rpy="0 0 0" xyz="0 0 0.0584" />
         <axis xyz="0 1 0" />
-        <limit effort="20" lower="0.0" upper="0.04" velocity="0.2" />
+        <limit effort="100" lower="0.0" upper="0.04" velocity="0.02" />
     </joint>
     <joint name="panda_finger_joint2" type="prismatic">
@@ -282,5 +282,5 @@
         <origin rpy="0 0 0" xyz="0 0 0.0584" />
         <axis xyz="0 -1 0" />
-        <limit effort="20" lower="0.0" upper="0.04" velocity="0.2" />
+        <limit effort="100" lower="0.0" upper="0.04" velocity="0.02" />
         <mimic joint="panda_finger_joint1" multiplier="1.0" offset="0.0"/>
     </joint>
@@ -330,4 +330,20 @@
         </joint>
     </ros2_control>
+    <gazebo reference="panda_leftfinger">
+      <mu1>10.0</mu1>
+      <mu2>10.0</mu2>
+      <kp>100000.0</kp>
+      <kd>10.0</kd>
+      <minDepth>0.005</minDepth>
+      <maxVel>0.001</maxVel>
+    </gazebo>
+    <gazebo reference="panda_rightfinger">
+      <mu1>10.0</mu1>
+      <mu2>10.0</mu2>
+      <kp>100000.0</kp>
+      <kd>10.0</kd>
+      <minDepth>0.005</minDepth>
+      <maxVel>0.001</maxVel>
+    </gazebo>
     <gazebo>
         <plugin filename="libgazebo_ros2_control.so" name="gazebo_ros2_control">
